File: hlk-pm-pcb.sch (KiCad schematic (older format))
At the start: 10 parts, among them J1 AC-In, J2 DC-Out

Commit message: development
Parts:
- F3: value Fuse -> Fuse 1.5A
Changed lines of the file:
@@
 P 6450 3850
 F 0 "F3" V 6253 3850 50  0000 C CNN
-F 1 "Fuse" V 6344 3850 50  0000 C CNN
+F 1 "Fuse 1.5A" V 6344 3850 50  0000 C CNN
 F 2 "Fuse:Fuse_1206_3216Metric" V 6380 3850 50  0001 C CNN
 F 3 "~" H 6450 3850 50  0001 C CNN

Commit message: Release board v.1.0
Parts:
- C1: Description (none) -> Capacitor 0.1 uF SMD 0805; Link (none) -> https://lcsc.com/product-detail/Multilayer-Ceramic-Capacito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; MOQ (none) -> 50; MPN (none) -> 0805B104K500NT; Manufacturer (none) -> FH(Guangdong Fenghua Advanced Tech); Price (none) -> 0.0043; VPN (none) -> C38141; Vendor (none) -> LCSC
- C2: Description (none) -> Capacitor 220 uF SMD; Link (none) -> https://lcsc.com/product-detail/Aluminum-Electrolytic-Capac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; MOQ (none) -> 5; MPN (none) -> CS1E221M-CRF10; Manufacturer (none) -> ST(Semtech); Price (none) -> 0.0786; VPN (none) -> C97815; Vendor (none) -> LCSC
- F1: Description (none) -> 5x20 mm fuse holder; Link (none) -> https://lcsc.com/product-detail/Fuse-Holders_Xucheng-Elec-C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; MOQ (none) -> 1; MPN (none) -> C58066; Manufacturer (none) -> Xucheng Elec; Price (none) -> 0.16; VPN (none) -> C58066; Vendor (none) -> LCSC
- F2: Description (none) -> Thermal Cutoff - 77°C; Link (none) -> https://lcsc.com/product-detail/Thermal-Cutoffs-TCO_Better-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; MOQ (none) -> 1; MPN (none) -> BTT010077; Manufacturer (none) -> Better; Price (none) -> 0.19; VPN (none) -> C723282; Vendor (none) -> LCSC
- F3: Description (none) -> Fuse 1.5A - SMD 1206; Link (none) -> https://lcsc.com/product-detail/Fuses_Shenzhen-lanson-Elec-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; MPN (none) -> 12D1150C; Manufacturer (none) -> Shenzhen lanson Elec; VPN (none) -> C182307; Vendor (none) -> LCSC
- J1, J2: Description (none) -> Screw terminal 2 pin p.5.08; Link (none) -> https://lcsc.com/product-detail/New-Quadratic-Unclassified-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; MOQ (none) -> 5; MPN (none) -> KF127-5.08-2P; Manufacturer (none) -> Cixi Kefa Elec; Price (none) -> 0.1311; VPN (none) -> C474906; Vendor (none) -> LCSC
- JP1: Description (none) -> Solder Jumper (no components required); Link (none) -> NA; MOQ (none) -> NA; MPN (none) -> NA; Manufacturer (none) -> NA; Price (none) -> NA; VPN (none) -> NA; Vendor (none) -> NA
- PS1: Description (none) -> AC-DC converter module; Link (none) -> https://lcsc.com/product-detail/Power-Modules_HI-LINK-HLK-P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; MOQ (none) -> 1; MPN (none) -> HLK-PM03; Manufacturer (none) -> HI-LINK; Price (none) -> 3.08; VPN (none) -> C209904; Vendor (none) -> LCSC
- RV1: Description (none) -> Varistor 510V VDR-10D511K; Link (none) -> https://lcsc.com/product-detail/Varistors_VDR-Varistor-VDR-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; MOQ (none) -> 10; MPN (none) -> VDR-10D511K; Manufacturer (none) -> VDR-Varistor; Price (none) -> 0.0458; VPN (none) -> C273559; Vendor (none) -> LCSC
Connections:
- net at PS1.2 (AC/N), RV1.2: now also J1.2 (Pin_2); no longer J1.1 (Pin_1)
- net at F1.2: now also J1.1 (Pin_1); no longer J1.2 (Pin_2)
- net at C1.2, C2.2, PS1.3 (-Vout): now also J2.1 (Pin_1); no longer J2.2 (Pin_2)
- net at C1.1, C2.1, F3.1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: now also J2.2 (Pin_2); no longer J2.1 (Pin_1)
Changed lines of the file:
@@
 encoding utf-8
 Sheet 1 1
-Title "HLC-PM-pcb"
+Title "HLK-PM-pcb"
 Date "2022-01-06"
 Rev "1.0"
@@
 L Connector:Screw_Terminal_01x02 J1
 U 1 1 61D77D19
-P 2850 3950
-F 0 "J1" H 2768 3625 50  0000 C CNN
-F 1 "AC-In" H 2768 3716 50  0000 C CNN
-F 2 "TerminalBlock:TerminalBlock_bornier-2_P5.08mm" H 2850 3950 50  0001 C CNN
-F 3 "~" H 2850 3950 50  0001 C CNN
-	1    2850 3950
-	-1   0    0    1
+P 2850 3850
+F 0 "J1" H 2768 3525 50  0000 C CNN
+F 1 "AC-In" H 2768 3616 50  0000 C CNN
+F 2 "TerminalBlock:TerminalBlock_bornier-2_P5.08mm" H 2850 3850 50  0001 C CNN
+F 3 "~" H 2850 3850 50  0001 C CNN
+F 4 "Screw terminal 2 pin p.5.08" H 2850 3850 50  0001 C CNN "Description"
+F 5 "https://lcsc.com/product-detail/New-Quadratic-Unclassified-Data_Cixi-Kefa-Elec-KF127-5-08-2P_C474906.html" H 2850 3850 50  0001 C CNN "Link"
+F 6 "5" H 2850 3850 50  0001 C CNN "MOQ"
+F 7 "KF127-5.08-2P" H 2850 3850 50  0001 C CNN "MPN"
+F 8 "Cixi Kefa Elec" H 2850 3850 50  0001 C CNN "Manufacturer"
+F 9 "0.1311" H 2850 3850 50  0001 C CNN "Price"
+F 10 "C474906" H 2850 3850 50  0001 C CNN "VPN"
+F 11 "LCSC" H 2850 3850 50  0001 C CNN "Vendor"
+	1    2850 3850
+	-1   0    0    -1
 $EndComp
 $Comp
@@
 F 2 "Converter_ACDC:Converter_ACDC_HiLink_HLK-PMxx" H 5700 3650 50  0001 C CNN
 F 3 "http://www.hlktech.net/product_detail.php?ProId=59" H 6100 3600 50  0001 C CNN
+F 4 "https://lcsc.com/product-detail/Power-Modules_HI-LINK-HLK-PM03_C209904.html" H 5700 3950 50  0001 C CNN "Link"
+F 5 "1" H 5700 3950 50  0001 C CNN "MOQ"
+F 6 "HLK-PM03" H 5700 3950 50  0001 C CNN "MPN"
+F 7 "HI-LINK" H 5700 3950 50  0001 C CNN "Manufacturer"
+F 8 "C209904" H 5700 3950 50  0001 C CNN "VPN"
+F 9 "LCSC" H 5700 3950 50  0001 C CNN "Vendor"
+F 10 "AC-DC converter module" H 5700 3950 50  0001 C CNN "Description"
+F 11 "3.08" H 5700 3950 50  0001 C CNN "Price"
 	1    5700 3950
 	1    0    0    -1
@@
 F 2 "Fuse:Fuseholder_Cylinder-5x20mm_Schurter_0031_8201_Horizontal_Open" V 3480 3850 50  0001 C CNN
 F 3 "~" H 3550 3850 50  0001 C CNN
+F 4 "LCSC" H 3550 3850 50  0001 C CNN "Vendor"
+F 5 "5x20 mm fuse holder" H 3550 3850 50  0001 C CNN "Description"
+F 6 "https://lcsc.com/product-detail/Fuse-Holders_Xucheng-Elec-C58066_C58066.html" H 3550 3850 50  0001 C CNN "Link"
+F 7 "1" H 3550 3850 50  0001 C CNN "MOQ"
+F 8 "C58066" H 3550 3850 50  0001 C CNN "MPN"
+F 9 "Xucheng Elec" H 3550 3850 50  0001 C CNN "Manufacturer"
+F 10 "0.16" H 3550 3850 50  0001 C CNN "Price"
+F 11 "C58066" H 3550 3850 50  0001 C CNN "VPN"
 	1    3550 3850
 	0    1    1    0
@@
 F 2 "Varistor:RV_Disc_D12mm_W6.2mm_P7.5mm" V 4730 4000 50  0001 C CNN
 F 3 "~" H 4800 4000 50  0001 C CNN
+F 4 "Varistor  510V VDR-10D511K" H 4800 4000 50  0001 C CNN "Description"
+F 5 "https://lcsc.com/product-detail/Varistors_VDR-Varistor-VDR-10D511K_C273559.html" H 4800 4000 50  0001 C CNN "Link"
+F 6 "10" H 4800 4000 50  0001 C CNN "MOQ"
+F 7 "VDR-10D511K" H 4800 4000 50  0001 C CNN "MPN"
+F 8 "VDR-Varistor" H 4800 4000 50  0001 C CNN "Manufacturer"
+F 9 "0.0458" H 4800 4000 50  0001 C CNN "Price"
+F 10 "C273559" H 4800 4000 50  0001 C CNN "VPN"
+F 11 "LCSC" H 4800 4000 50  0001 C CNN "Vendor"
 	1    4800 4000
 	1    0    0    -1
@@
 L Connector:Screw_Terminal_01x02 J2
 U 1 1 61D7D6E4
-P 8000 3850
-F 0 "J2" H 8080 3842 50  0000 L CNN
-F 1 "DC-Out" H 8080 3751 50  0000 L CNN
-F 2 "TerminalBlock:TerminalBlock_bornier-2_P5.08mm" H 8000 3850 50  0001 C CNN
-F 3 "~" H 8000 3850 50  0001 C CNN
-	1    8000 3850
-	1    0    0    -1
+P 8000 3950
+F 0 "J2" H 8080 3942 50  0000 L CNN
+F 1 "DC-Out" H 8080 3851 50  0000 L CNN
+F 2 "TerminalBlock:TerminalBlock_bornier-2_P5.08mm" H 8000 3950 50  0001 C CNN
+F 3 "~" H 8000 3950 50  0001 C CNN
+F 4 "Screw terminal 2 pin p.5.08" H 8000 3950 50  0001 C CNN "Description"
+F 5 "https://lcsc.com/product-detail/New-Quadratic-Unclassified-Data_Cixi-Kefa-Elec-KF127-5-08-2P_C474906.html" H 8000 3950 50  0001 C CNN "Link"
+F 6 "5" H 8000 3950 50  0001 C CNN "MOQ"
+F 7 "KF127-5.08-2P" H 8000 3950 50  0001 C CNN "MPN"
+F 8 "Cixi Kefa Elec" H 8000 3950 50  0001 C CNN "Manufacturer"
+F 9 "0.1311" H 8000 3950 50  0001 C CNN "Price"
+F 10 "C474906" H 8000 3950 50  0001 C CNN "VPN"
+F 11 "LCSC" H 8000 3950 50  0001 C CNN "Vendor"
+	1    8000 3950
+	1    0    0    1
 $EndComp
 $Comp
@@
 F 2 "Capacitor_SMD:C_0805_2012Metric" H 6838 3850 50  0001 C CNN
 F 3 "~" H 6800 4000 50  0001 C CNN
+F 4 "Capacitor 0.1 uF SMD 0805" H 6800 4000 50  0001 C CNN "Description"
+F 5 "https://lcsc.com/product-detail/Multilayer-Ceramic-Capacitors-MLCC-SMD-SMT_100nF-104-10-50V_C38141.html" H 6800 4000 50  0001 C CNN "Link"
+F 6 "50" H 6800 4000 50  0001 C CNN "MOQ"
+F 7 "0805B104K500NT" H 6800 4000 50  0001 C CNN "MPN"
+F 8 "FH(Guangdong Fenghua Advanced Tech)" H 6800 4000 50  0001 C CNN "Manufacturer"
+F 9 "0.0043" H 6800 4000 50  0001 C CNN "Price"
+F 10 "C38141" H 6800 4000 50  0001 C CNN "VPN"
+F 11 "LCSC" H 6800 4000 50  0001 C CNN "Vendor"
 	1    6800 4000
 	1    0    0    -1
@@
 F 2 "Capacitor_SMD:CP_Elec_8x10.5" H 7300 4000 50  0001 C CNN
 F 3 "~" H 7300 4000 50  0001 C CNN
+F 4 "Capacitor 220 uF SMD" H 7300 4000 50  0001 C CNN "Description"
+F 5 "https://lcsc.com/product-detail/Aluminum-Electrolytic-Capacitors-SMD_ST-Semtech-CS1E221M-CRF10_C97815.html" H 7300 4000 50  0001 C CNN "Link"
+F 6 "5" H 7300 4000 50  0001 C CNN "MOQ"
+F 7 "CS1E221M-CRF10" H 7300 4000 50  0001 C CNN "MPN"
+F 8 "ST(Semtech)" H 7300 4000 50  0001 C CNN "Manufacturer"
+F 9 "0.0786" H 7300 4000 50  0001 C CNN "Price"
+F 10 "C97815" H 7300 4000 50  0001 C CNN "VPN"
+F 11 "LCSC" H 7300 4000 50  0001 C CNN "Vendor"
 	1    7300 4000
 	1    0    0    -1
@@
 F 2 "Resistor_THT:R_Axial_DIN0516_L15.5mm_D5.0mm_P25.40mm_Horizontal" V 4380 3850 50  0001 C CNN
 F 3 "~" H 4450 3850 50  0001 C CNN
+F 4 "Thermal Cutoff - 77°C" H 4450 3850 50  0001 C CNN "Description"
+F 5 "https://lcsc.com/product-detail/Thermal-Cutoffs-TCO_Better-BTT010077_C723282.html" H 4450 3850 50  0001 C CNN "Link"
+F 6 "1" H 4450 3850 50  0001 C CNN "MOQ"
+F 7 "BTT010077" H 4450 3850 50  0001 C CNN "MPN"
+F 8 "Better" H 4450 3850 50  0001 C CNN "Manufacturer"
+F 9 "0.19" H 4450 3850 50  0001 C CNN "Price"
+F 10 "C723282" H 4450 3850 50  0001 C CNN "VPN"
+F 11 "LCSC" H 4450 3850 50  0001 C CNN "Vendor"
 	1    4450 3850
 	0    1    1    0
@@
 F 2 "Fuse:Fuse_1206_3216Metric" V 6380 3850 50  0001 C CNN
 F 3 "~" H 6450 3850 50  0001 C CNN
+F 4 "Fuse 1.5A - SMD 1206" H 6450 3850 50  0001 C CNN "Description"
+F 5 "https://lcsc.com/product-detail/Fuses_Shenzhen-lanson-Elec-12D1150C_C182307.html" H 6450 3850 50  0001 C CNN "Link"
+F 6 "12D1150C" H 6450 3850 50  0001 C CNN "MPN"
+F 7 "Shenzhen lanson Elec" H 6450 3850 50  0001 C CNN "Manufacturer"
+F 8 "C182307" H 6450 3850 50  0001 C CNN "VPN"
+F 9 "LCSC" H 6450 3850 50  0001 C CNN "Vendor"
 	1    6450 3850
 	0    1    1    0
@@
 F 2 "Jumper:SolderJumper-2_P1.3mm_Open_TrianglePad1.0x1.5mm" H 6450 3400 50  0001 C CNN
 F 3 "~" H 6450 3400 50  0001 C CNN
+F 4 "Solder Jumper (no components required)" H 6450 3400 50  0001 C CNN "Description"
+F 5 "NA" H 6450 3400 50  0001 C CNN "Link"
+F 6 "NA" H 6450 3400 50  0001 C CNN "MOQ"
+F 7 "NA" H 6450 3400 50  0001 C CNN "MPN"
+F 8 "NA" H 6450 3400 50  0001 C CNN "Manufacturer"
+F 9 "NA" H 6450 3400 50  0001 C CNN "Price"
+F 10 "NA" H 6450 3400 50  0001 C CNN "VPN"
+F 11 "NA" H 6450 3400 50  0001 C CNN "Vendor"
 	1    6450 3400
 	1    0    0    -1
